File: Rev A/SurgicalLightBatteryModule.kicad_pcb (KiCad board)
At the start: 2 copper layers, 0 parts

Commit message: Updated PCB and Schematics
Parts:
- added C1: 0.1uF, Capacitor_SMD:C_0805_2012Metric, F.Cu at (166.0, 119.3)
- added C2: 470uF, Capacitor_SMD:C_0805_2012Metric_Pad1.18x1.45mm_HandSolder, F.Cu at (169.1, 119.4)
- added C3: 470uF, Capacitor_SMD:C_0805_2012Metric_Pad1.18x1.45mm_HandSolder, F.Cu at (172.2, 119.4)
- added C4: 0.1uF, Capacitor_SMD:C_0805_2012Metric, F.Cu at (177.7, 101.5)
- added C5: 1nF, Capacitor_SMD:C_0805_2012Metric_Pad1.18x1.45mm_HandSolder, F.Cu at (145.3, 89.0)
- added C6: 100nF, Capacitor_SMD:C_0805_2012Metric_Pad1.18x1.45mm_HandSolder, F.Cu at (141.9, 83.8)
- added C7: 22uF, Capacitor_SMD:C_0805_2012Metric_Pad1.18x1.45mm_HandSolder, F.Cu at (183.6, 95.4)
- added C8: 0.1uF, Capacitor_SMD:C_0805_2012Metric, F.Cu at (183.5, 92.2)
- added D1: PMEG045V150EPD, Package_TO_SOT_SMD:Nexperia_CFP15_SOT-1289, F.Cu at (160.9, 117.1)
- added D2: PMEG045V150EPD, Package_TO_SOT_SMD:Nexperia_CFP15_SOT-1289, F.Cu at (178.8, 111.1)
- added D3: PMEG045V150EPD, Package_TO_SOT_SMD:Nexperia_CFP15_SOT-1289, F.Cu at (177.6, 95.6)
- added D4: SZSMF4L15CAT3G, Diode_SMD:D_SOD-123F, F.Cu at (183.7, 97.9)
- added D5: LED, Diode_SMD:D_3220_8050Metric_Pad2.65x5.15mm_HandSolder, F.Cu at (182.2, 73.1)
- added D6: 1N4148, Diode_THT:D_DO-35_SOD27_P7.62mm_Horizontal, F.Cu at (195.6, 78.7)
- added D7: LED Green, LED_SMD:LED_0805_2012Metric, F.Cu at (174.8, 88.4)
- added F1: 12A, Fuse:Fuse_0805_2012Metric_Pad1.15x1.40mm_HandSolder, F.Cu at (183.8, 88.3)
- added F2: 10A, Fuse:Fuse_0805_2012Metric_Pad1.15x1.40mm_HandSolder, F.Cu at (141.8, 70.7)
- added L1: 100uH 10.5A, Inductor_SMD:L_0805_2012Metric, F.Cu at (183.8, 101.0)
- added Q1: BC337, Package_TO_SOT_THT:TO-92_Inline, F.Cu at (169.6, 96.2)
- added Q2: IRLZ44N, Package_TO_SOT_THT:TO-220-3_Vertical, F.Cu at (166.5, 107.6)
- added Q3: BC557, Package_TO_SOT_THT:TO-92_Inline, F.Cu at (177.8, 83.8)
- added Q4: BC327, Package_TO_SOT_THT:TO-92_Inline, F.Cu at (169.6, 101.3)
- added Q5: IRLZ44N, Package_TO_SOT_THT:TO-220-3_Vertical, F.Cu at (166.5, 113.8)
- added R1: 10K, Resistor_SMD:R_0805_2012Metric_Pad1.20x1.40mm_HandSolder, F.Cu at (138.8, 75.5)
- added R12: 0R1, Resistor_SMD:R_0805_2012Metric_Pad1.20x1.40mm_HandSolder, F.Cu at (155.3, 64.5)
- added R13: 2K, Resistor_SMD:R_0805_2012Metric_Pad1.20x1.40mm_HandSolder, F.Cu at (159.2, 62.4)
- added R14: 2K, Resistor_SMD:R_0805_2012Metric_Pad1.20x1.40mm_HandSolder, F.Cu at (156.8, 68.9)
- added R15: 47K, Resistor_SMD:R_0805_2012Metric_Pad1.20x1.40mm_HandSolder, F.Cu at (160.5, 68.7)
- added R16: 47K, Resistor_SMD:R_0805_2012Metric_Pad1.20x1.40mm_HandSolder, F.Cu at (155.4, 59.9)
- added R18: 10K, Resistor_SMD:R_0805_2012Metric_Pad1.20x1.40mm_HandSolder, F.Cu at (168.5, 75.5)
- added R19: 10K, Resistor_SMD:R_0805_2012Metric_Pad1.20x1.40mm_HandSolder, F.Cu at (174.0, 75.5)
- added R2: 2.2K, Resistor_SMD:R_0805_2012Metric_Pad1.20x1.40mm_HandSolder, F.Cu at (144.2, 75.3)
- added R20: 39K, Resistor_SMD:R_0805_2012Metric_Pad1.20x1.40mm_HandSolder, F.Cu at (145.3, 91.6)
- added R21: 2K2, Resistor_SMD:R_0805_2012Metric_Pad1.20x1.40mm_HandSolder, F.Cu at (187.8, 67.3)
- added R22: 10K, Resistor_SMD:R_0805_2012Metric_Pad1.20x1.40mm_HandSolder, F.Cu at (192.1, 67.1)
- added R23: 2K, Resistor_SMD:R_0805_2012Metric_Pad1.20x1.40mm_HandSolder, F.Cu at (197.2, 67.0)
- added R24: 2K2, Resistor_SMD:R_0805_2012Metric_Pad1.20x1.40mm_HandSolder, F.Cu at (183.9, 83.8)
- added R25: 10K, Resistor_SMD:R_0805_2012Metric_Pad1.20x1.40mm_HandSolder, F.Cu at (183.9, 81.3)
- added R26: 47K, Resistor_SMD:R_0805_2012Metric_Pad1.20x1.40mm_HandSolder, F.Cu at (137.8, 83.0)
- added R27: 56k, Resistor_SMD:R_0805_2012Metric_Pad1.20x1.40mm_HandSolder, F.Cu at (146.0, 82.7)
- added R28: 10K, Resistor_SMD:R_0805_2012Metric_Pad1.20x1.40mm_HandSolder, F.Cu at (140.0, 88.2)
- added R29: 1K, Resistor_SMD:R_0805_2012Metric_Pad1.20x1.40mm_HandSolder, F.Cu at (134.0, 88.2)
- added R3: 2k2, Resistor_SMD:R_0805_2012Metric, F.Cu at (168.8, 92.0)
- added R30: 10K, Resistor_SMD:R_0805_2012Metric_Pad1.20x1.40mm_HandSolder, F.Cu at (136.6, 88.3)
- added R4: 5, Resistor_SMD:R_0805_2012Metric, F.Cu at (164.0, 102.4)
- added R5: 1K, Resistor_SMD:R_0805_2012Metric, F.Cu at (179.2, 88.5)
- added R7: 560R, Resistor_SMD:R_0805_2012Metric_Pad1.20x1.40mm_HandSolder, F.Cu at (153.7, 69.0)
- added RV2: 10K, Potentiometer_THT:Potentiometer_Bourns_3339P_Vertical_HandSoldering, F.Cu at (149.9, 59.8)
- added U1: TL494, Package_DIP:DIP-16_W7.62mm_Socket, F.Cu at (156.4, 74.7)
- added U2: LM358, Package_DIP:DIP-8_W7.62mm_Socket, F.Cu at (163.6, 61.9)
- added U3: TL431D, Package_SO:SOIC-8_3.9x4.9mm_P1.27mm, F.Cu at (190.2, 72.7)
Routing:
- net GND: track 0.00 -> 103.5 mm, vias 0 -> 7
- net /battery_module_analog/VREF: track 0.00 -> 81.3 mm
- net BAT+: track 0.00 -> 52.3 mm, vias 0 -> 2
- net Net-(D3-K): track 0.00 -> 32.6 mm
- net Net-(D1-K): track 0.00 -> 32.1 mm
- net /battery_module_analog/EA1-: track 0.00 -> 31.6 mm
- net Net-(D2-K): track 0.00 -> 29.0 mm, vias 0 -> 2
- net /battery_module_analog/VPOut: track 0.00 -> 27.2 mm
- net /battery_module_analog/EA2+: track 0.00 -> 20.9 mm
- net Net-(D5-K): track 0.00 -> 20.6 mm
- net /battery_module_analog/EA1+: track 0.00 -> 18.4 mm
- net /battery_module_power/PWM Out: track 0.00 -> 17.7 mm
- net Net-(R16-Pad1): track 0.00 -> 16.0 mm
- net /battery_module_analog/FB: track 0.00 -> 15.1 mm
- net Net-(D6-A): track 0.00 -> 13.5 mm
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- added copper zone on F.Cu, net GND
Other:
- board outline added: 76.2 x 76.2 mm
- board text added: "Buck Section"
- board text added: "Inputs Power Module"
- board text added: "Oscillation Frequency parameters"
- board text added: "Power Output"
