File: Rev A/SurgicalLightBatteryModule.kicad_pcb (KiCad board)
At the start: 2 copper layers, 76.2 x 76.2 mm, 51 parts, among them Q1 BC337, Q2 IRLZ44N, Q3 BC557, Q4 BC327, Q5 IRLZ44N, U1 TL494, U2 LM358, U3 TL431D

Commit message: Battery Module (04/01/2024)
Parts:
- added REF**: MountingHole_2.5mm, MountingHole:MountingHole_2.5mm, F.Cu at (132.1, 55.9)
- added REF**: MountingHole_2.5mm, MountingHole:MountingHole_2.5mm, F.Cu at (198.1, 121.9)
- added REF**: MountingHole_2.5mm, MountingHole:MountingHole_2.5mm, F.Cu at (132.1, 121.9)
- added REF**: MountingHole_2.5mm, MountingHole:MountingHole_2.5mm, F.Cu at (198.1, 55.9)
Other:
- board text removed: "Buck Section"
- board text removed: "Inputs Power Module"
- board text removed: "Oscillation Frequency parameters"
- board text removed: "Power Output"
