File: Version-04-03-2024/Version-04-03-2024.kicad_pcb (KiCad board)
At the start: 2 copper layers, 58 parts, among them Q3 BC337, Q6 BC557, Q7 IRLZ44N, Q8 BC327, Q9 IRLZ44N, U4 TL494, U5 LM358, U6 TL431D

Commit message: Update 04/05
Parts:
- removed REF** (x4): MountingHole_3mm, MountingHole:MountingHole_3mm
- added H1: M3 Hole, MountingHole:MountingHole_3.2mm_M3_Pad_TopBottom, F.Cu at (212.1, 74.9)
- added H2: M3 Hole, MountingHole:MountingHole_3.2mm_M3_Pad_TopBottom, F.Cu at (87.6, 74.9)
- added H3: M3 Hole, MountingHole:MountingHole_3.2mm_M3_Pad_TopBottom, F.Cu at (87.6, 55.9)
- added H4: M3 Hole, MountingHole:MountingHole_3.2mm_M3_Pad_TopBottom, F.Cu at (212.1, 55.9)
- added J1: Conn_01x01_Pin, Connector_PinHeader_2.54mm:PinHeader_1x01_P2.54mm_Vertical, F.Cu at (127.0, 59.7)
- moved F2 103.0 mm to (130.8, 125.7), turned to 180 degrees
- moved D12 90.6 mm to (129.2, 86.4), turned to 180 degrees
- moved R7 89.1 mm to (129.2, 90.2)
- moved D3 51.3 mm to (162.8, 119.4)
- moved Q8 40.2 mm to (144.8, 95.2)
- moved C12 39.3 mm to (148.6, 89.8)
- moved C6 38.9 mm to (198.1, 82.5), turned to -90 degrees
- moved D2 38.3 mm to (162.8, 109.2)
- moved Q3 36.3 mm to (144.1, 88.9)
- moved C7 34.5 mm to (181.6, 82.5), turned to -90 degrees
- moved D11 29.8 mm to (189.4, 128.3), turned to 180 degrees
- moved RV1 27.9 mm to (170.2, 72.4)
- moved D1 25.5 mm to (163.2, 100.1)
- moved Q9 24.7 mm to (151.7, 102.9), turned to -90 degrees
- moved C14 24.2 mm to (162.6, 127.0), turned to 90 degrees
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Connections:
- D5 pad 1: BatteryModuleVin -> SOLAR+
- D5 pad 2: BatteryModuleVin -> SOLAR+
- F2 pad 2: VBattery -> BAT+
- R37 pad 2: Net-(R37-Pad2) -> GND
- R39 pad 1: Net-(R37-Pad2) -> GND
- R7 pad 1: VBattery -> BAT+
Routing:
- net GND: track 0.00 -> 80.0 mm, vias 0 -> 15
- net /VREF: track 0.00 -> 45.7 mm
- net Net-(F3-Pad1): track 0.00 -> 42.0 mm
- net /EA2+: track 0.00 -> 34.5 mm
- net /PWM Out: track 0.00 -> 29.9 mm
- net MCU 2.5V: track 0.00 -> 25.3 mm
- net Net-(Q7-G): track 0.00 -> 23.4 mm, vias 0 -> 1
- net /VPOut: track 0.00 -> 19.7 mm
- net Net-(D6-K): track 0.00 -> 19.1 mm
- net Net-(D8-A): track 0.00 -> 16.6 mm
- net Net-(D9-A): track 0.00 -> 15.9 mm
- net /EA1-: track 0.00 -> 15.8 mm
- net Net-(D8-K): track 0.00 -> 14.5 mm
- net /CT: track 0.00 -> 13.0 mm
- net Net-(Q3-E): track 0.00 -> 12.9 mm
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- added copper zone on F.Cu, net BAT+
- added copper zone on F.Cu, net BAT-
- added copper zone on B.Cu, net GND
- added copper zone on F.Cu, net Net-(D1-K)
- added copper zone on F.Cu, net Net-(D11-A2)
- added copper zone on F.Cu, net Net-(D5-K)
- added copper zone on F.Cu, net SOLAR+
