File: Version-04-03-2024/Version-04-03-2024.kicad_sch (KiCad schematic)
At the start: 54 parts, among them Q3 BC337, Q6 BC557, Q7 IRLZ44N, Q8 BC327, Q9 IRLZ44N, U4 TL494, U5 LM358, U6 TL431D

Commit message: Update 04/05
Parts:
- added H1, H2, H3, H4: M3 Hole, MountingHole:MountingHole_3.2mm_M3_Pad_TopBottom, symbol Mechanical:MountingHole_Pad
- added J1: Conn_01x01_Pin, Connector_PinHeader_2.54mm:PinHeader_1x01_P2.54mm_Vertical, symbol Connector:Conn_01x01_Pin
Connections:
- net BatteryModuleVin is gone; now on net SOLAR+: D5.1 (A), D5.2 (A)
- net VBattery is gone; now on net BAT+: F2.2, R7.1
- net BAT+: now also H3.1
- net BAT-: now also H4.1
- net GND: now also R37.2, R39.1, H2.1
- net MCU 2.5V: now also J1.1 (Pin_1)
- net SOLAR+: now also H1.1
Other:
- note added: "Battery/Power Holes"
- note added: "Header Connection (MCU Input)"
